File: pcb/revB/ma42_PCB_revB/keyboard.kicad_pcb (KiCad board)
At the start: 2 copper layers, 241.8 x 75.2 mm, 107 parts, among them IC1 ATMEGA32U4, J1 MINI, J2 USBMINI_B05, X1 ASX3F

Commit message: working on revB
Parts:
- added D45: 1N4148, SM0805D_big, B.Cu at (314.5, 150.6)
- added S46: Reset, DTSJW-66N, B.Cu at (242.8, 142.7)
- C4: value 22p -> 100n
- C6: value 100n -> 22p
- J1: value MINI -> USB
- J2: value USBMINI_B05 -> USB
- S1: value DTSM-6 -> MX1A; footprint DTSJW-66N -> MX1A-b; moved to F.Cu
- moved S1 143.1 mm to (99.8, 87.6)
- moved S37 63.7 mm to (280.8, 144.8)
- moved D33 63.5 mm to (254.8, 150.6)
- moved S5 61.7 mm to (118.9, 87.6)
- moved S9 60.9 mm to (137.9, 87.6)
- moved D20 60.4 mm to (190.5, 93.5)
- moved S13 60.1 mm to (157.0, 87.6)
- moved D29 59.1 mm to (221.2, 150.6)
- moved S17 57.3 mm to (176.0, 87.6)
- moved C6 52.9 mm to (215.9, 138.2), turned to 180 degrees
- moved D24 49.2 mm to (214.4, 112.5)
- moved D25 48.3 mm to (219.2, 131.6)
- moved D36 47.6 mm to (276.4, 131.6)
- moved S22 47.3 mm to (204.6, 125.7)
- moved S40 47.3 mm to (299.8, 125.7)
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Connections:
- C4 pad 1: N-0000035 -> VCC
- C6 pad 1: VCC -> N-0000035
- D1 pad 2: N-0000044 -> N-0000043
- D10 pad 2: N-0000058 -> N-0000063
- D11 pad 2: N-0000057 -> N-0000061
- D12 pad 2: N-0000055 -> N-0000059
- D13 pad 2: N-0000064 -> N-0000070
- D14 pad 2: N-0000067 -> N-0000069
- D15 pad 2: N-0000066 -> N-0000068
- D16 pad 2: N-0000065 -> N-0000067
- D17 pad 2: N-0000043 -> N-0000048
- D18 pad 2: N-0000048 -> N-0000054
- D19 pad 2: N-0000045 -> N-0000042
- D2 pad 2: N-0000061 -> N-0000066
- D20 pad 1: /Matrix/col9 -> /Matrix/col6
- D20 pad 2: N-0000074 -> N-0000058
- D21 pad 2: N-0000071 -> N-0000062
- D22 pad 2: N-0000070 -> N-0000072
- D23 pad 1: /Matrix/col6 -> /Matrix/col7
- D23 pad 2: N-0000069 -> N-0000047
- D24 pad 1: /Matrix/col10 -> /Matrix/col7
- D24 pad 2: N-0000068 -> N-0000046
- D25 pad 2: N-0000042 -> N-0000045
- D26 pad 1: /Matrix/col7 -> /Matrix/col8
- D26 pad 2: N-0000054 -> N-0000044
- D27 pad 1: /Matrix/col7 -> /Matrix/col8
- D27 pad 2: N-0000050 -> N-0000056
- D28 pad 1: /Matrix/col11 -> /Matrix/col8
- D28 pad 2: N-0000085 -> N-0000055
- D29 pad 2: N-0000053 -> N-0000075
- D3 pad 2: N-0000073 -> N-0000074
- D30 pad 1: /Matrix/col8 -> /Matrix/col9
- D30 pad 2: N-0000051 -> N-0000057
- D31 pad 1: /Matrix/col8 -> /Matrix/col9
- D31 pad 2: N-0000049 -> N-0000052
- D32 pad 1: /Matrix/col12 -> /Matrix/col9
- D32 pad 2: N-0000084 -> N-0000053
- D33 pad 2: N-0000052 -> N-0000078
- D34 pad 1: /Matrix/col9 -> /Matrix/col10
- D34 pad 2: N-0000046 -> N-0000051
- D35 pad 1: /Matrix/col9 -> /Matrix/col10
- D35 pad 2: N-0000047 -> N-0000050
- D37 pad 2: N-0000082 -> N-0000071
- D38 pad 1: /Matrix/col10 -> /Matrix/col11
- D38 pad 2: N-0000079 -> N-0000049
- D39 pad 2: N-0000081 -> N-0000084
- D4 pad 2: N-0000072 -> N-0000073
- D40 pad 2: N-0000080 -> N-0000081
- D42 pad 2: N-0000075 -> N-0000079
- D43 pad 2: N-0000076 -> N-0000080
- D44 pad 2: N-0000078 -> N-0000082
- D5 pad 2: N-0000063 -> N-0000086
- D6 pad 2: N-0000060 -> N-0000065
- D7 pad 2: N-0000059 -> N-0000064
- D8 pad 2: N-0000056 -> N-0000060
- D9 pad 2: N-0000062 -> N-0000085
- S1 pad 1: GND -> /Matrix/row1
- S1 pad 2: (no net) -> N-0000043
- S10 pad 1: /Matrix/row1 -> /Matrix/row2
- S10 pad 2: N-0000062 -> N-0000063
- S11 pad 1: /Matrix/row2 -> /Matrix/row3
- S11 pad 2: N-0000058 -> N-0000061
- S12 pad 1: /Matrix/row3 -> /Matrix/row4
- S12 pad 2: N-0000057 -> N-0000059
- S13 pad 1: /Matrix/row4 -> /Matrix/row1
- S13 pad 2: N-0000055 -> N-0000070
- S14 pad 1: /Matrix/row1 -> /Matrix/row2
- S14 pad 2: N-0000064 -> N-0000069
- S15 pad 1: /Matrix/row2 -> /Matrix/row3
- S15 pad 2: N-0000067 -> N-0000068
- S16 pad 1: /Matrix/row3 -> /Matrix/row4
- S16 pad 2: N-0000066 -> N-0000067
- S17 pad 1: /Matrix/row4 -> /Matrix/row1
- S17 pad 2: N-0000065 -> N-0000048
- S18 pad 1: /Matrix/row1 -> /Matrix/row2
- S18 pad 2: N-0000043 -> N-0000054
- S19 pad 1: /Matrix/row2 -> /Matrix/row3
- S19 pad 2: N-0000048 -> N-0000042
- S2 pad 1: /Matrix/row1 -> /Matrix/row2
- S2 pad 2: N-0000044 -> N-0000066
- S20 pad 1: /Matrix/row3 -> /Matrix/row1
- S20 pad 2: N-0000045 -> N-0000058
- S21 pad 1: /Matrix/row4 -> /Matrix/row2
- S21 pad 2: N-0000074 -> N-0000062
- S22 pad 1: /Matrix/row1 -> /Matrix/row3
- S22 pad 2: N-0000071 -> N-0000072
- S23 pad 1: /Matrix/row2 -> /Matrix/row1
- S23 pad 2: N-0000070 -> N-0000047
- S24 pad 1: /Matrix/row3 -> /Matrix/row2
- S24 pad 2: N-0000069 -> N-0000046
- S25 pad 1: /Matrix/row4 -> /Matrix/row3
- S25 pad 2: N-0000068 -> N-0000045
- S26 pad 2: N-0000042 -> N-0000044
- S27 pad 2: N-0000054 -> N-0000056
- S28 pad 2: N-0000050 -> N-0000055
- S29 pad 2: N-0000085 -> N-0000075
- S3 pad 1: /Matrix/row2 -> /Matrix/row3
- S3 pad 2: N-0000061 -> N-0000074
- S30 pad 2: N-0000053 -> N-0000057
- S31 pad 2: N-0000051 -> N-0000052
- S32 pad 2: N-0000049 -> N-0000053
- S33 pad 2: N-0000084 -> N-0000078
- S34 pad 2: N-0000052 -> N-0000051
- S35 pad 2: N-0000046 -> N-0000050
- S36 pad 2: N-0000047 -> N-0000083
- S37 pad 1: /Matrix/row1 -> /Matrix/row4
- S37 pad 2: N-0000083 -> N-0000071
- S38 pad 1: /Matrix/row2 -> /Matrix/row1
- S38 pad 2: N-0000082 -> N-0000049
- S39 pad 1: /Matrix/row3 -> /Matrix/row2
- S39 pad 2: N-0000079 -> N-0000084
- S4 pad 1: /Matrix/row3 -> /Matrix/row4
- S40 pad 1: /Matrix/row1 -> /Matrix/row3
- S41 pad 1: /Matrix/row2 -> /Matrix/row4
- S41 pad 2: N-0000080 -> N-0000077
- S42 pad 1: /Matrix/row3 -> /Matrix/row1
- S42 pad 2: N-0000077 -> N-0000079
- S43 pad 1: /Matrix/row1 -> /Matrix/row2
- S43 pad 2: N-0000075 -> N-0000080
- S44 pad 1: /Matrix/row2 -> /Matrix/row3
- S44 pad 2: N-0000076 -> N-0000082
- S45 pad 1: /Matrix/row3 -> /Matrix/row4
- S45 pad 2: N-0000078 -> N-0000076
- S5 pad 1: /Matrix/row4 -> /Matrix/row1
- S5 pad 2: N-0000072 -> N-0000086
- S6 pad 1: /Matrix/row1 -> /Matrix/row2
- S6 pad 2: N-0000063 -> N-0000065
- S7 pad 1: /Matrix/row2 -> /Matrix/row3
- S7 pad 2: N-0000060 -> N-0000064
- S8 pad 1: /Matrix/row3 -> /Matrix/row4
- S8 pad 2: N-0000059 -> N-0000060
- S9 pad 1: /Matrix/row4 -> /Matrix/row1
- S9 pad 2: N-0000056 -> N-0000085
Routing:
- net /Matrix/row1: track 0.00 -> 334.1 mm, vias 0 -> 9
- net /Matrix/row2: track 0.00 -> 311.7 mm, vias 0 -> 3
- net /Matrix/row3: track 0.00 -> 292.1 mm, vias 0 -> 3
- net /Matrix/row4: track 0.00 -> 265.7 mm, vias 0 -> 1
- net N-0000031: track 0.00 -> 227.7 mm, vias 0 -> 4
- net N-0000026: track 0.00 -> 218.0 mm, vias 0 -> 3
- net /Matrix/col12: track 0.00 -> 173.9 mm, vias 0 -> 2
- net /Matrix/col1: track 0.00 -> 173.4 mm, vias 0 -> 2
- net /Matrix/col11: track 0.00 -> 159.9 mm, vias 0 -> 2
- net /Matrix/col2: track 0.00 -> 149.4 mm, vias 0 -> 2
- net /Matrix/col10: track 0.00 -> 142.3 mm, vias 0 -> 2
- net /Matrix/col3: track 0.00 -> 126.6 mm, vias 0 -> 2
- net /Matrix/col9: track 0.00 -> 122.6 mm, vias 0 -> 2
- net /Matrix/col8: track 0.00 -> 118.7 mm, vias 0 -> 2
- net /Matrix/col7: track 0.00 -> 103.8 mm, vias 0 -> 4
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- added copper zone on B.Cu, net GND
- added copper zone on F.Cu, net VCC
Other:
- board size 241.8 x 75.2 mm -> 236.7 x 74.7 mm
- board text added: "A 42% programmable keyboard designed for Dvorak."
- board text added: "Adam Schwartz & Michael Gobeli"
- board text added: "Inspired by the GH60, ErgoDox, and JD40."
- board text added: "revB"
- board text removed: "A programmable 42% keyboard for Dvorak."
- board text removed: "Adam Schwartz & Michael Gobeli Revision 2014-07-07"
- board text removed: "Inspired by: JD40, GH60 ErgoDox"
