File: pcb/revB/ma42_PCB_revB/keyboard.sch (KiCad schematic (older format))
At the start: 17 parts, among them IC1 ATMEGA32U4, J1 MINI, J2 USBMINI_B05, X1 ASX3F

Commit message: working on revB
Parts:
- renumbered C5 to C4, C6 to C5, C4 to C6, J2 to J1, J1 to J2, S1 to S46
Changed lines of the file:
@@
 Sheet 1 2
 Title "ukbdc - schematic"
-Date "19 jul 2014"
+Date "26 jul 2014"
 Rev ""
 Comp "komar"
@@
 $EndDescr
 $Comp
-L VCC #PWR01
+L VCC #PWR15
 U 1 1 4F085452
 P 4600 4550
-F 0 "#PWR01" H 4600 4650 30  0001 C CNN
+F 0 "#PWR15" H 4600 4650 30  0001 C CNN
 F 1 "VCC" H 4600 4650 30  0000 C CNN
 F 2 "" H 4600 4550 60  0001 C CNN
@@
 $EndComp
 $Comp
-L VCC #PWR02
+L VCC #PWR4
 U 1 1 4F08534F
 P 3300 5700
-F 0 "#PWR02" H 3300 5800 30  0001 C CNN
+F 0 "#PWR4" H 3300 5800 30  0001 C CNN
 F 1 "VCC" H 3300 5800 30  0000 C CNN
 F 2 "" H 3300 5700 60  0001 C CNN
@@
 NoConn ~ 3250 5050
 $Comp
-L USBMINI_B05 J1
+L USBMINI_B05 J2
 U 1 1 4F08252F
 P 3050 4950
-F 0 "J1" H 2975 5250 60  0000 C CNN
+F 0 "J2" H 2975 5250 60  0000 C CNN
 F 1 "MINI" H 3000 4600 60  0001 C CNN
 F 2 "" H 3050 4950 60  0001 C CNN
@@
 $EndComp
 $Comp
-L GND #PWR03
+L GND #PWR10
 U 1 1 4F08176B
 P 4100 3550
-F 0 "#PWR03" H 4100 3550 30  0001 C CNN
+F 0 "#PWR10" H 4100 3550 30  0001 C CNN
 F 1 "GND" H 4100 3480 30  0001 C CNN
 F 2 "" H 4100 3550 60  0001 C CNN
@@
 $EndComp
 $Comp
-L GND #PWR04
+L GND #PWR9
 U 1 1 4F081769
 P 3900 3550
-F 0 "#PWR04" H 3900 3550 30  0001 C CNN
+F 0 "#PWR9" H 3900 3550 30  0001 C CNN
 F 1 "GND" H 3900 3480 30  0001 C CNN
 F 2 "" H 3900 3550 60  0001 C CNN
@@
 $EndComp
 $Comp
-L GND #PWR05
+L GND #PWR3
 U 1 1 4ED6BB30
 P 2800 2600
-F 0 "#PWR05" H 2800 2600 30  0001 C CNN
+F 0 "#PWR3" H 2800 2600 30  0001 C CNN
 F 1 "GND" H 2800 2530 30  0001 C CNN
 F 2 "" H 2800 2600 60  0001 C CNN
@@
 $EndComp
 $Comp
-L VCC #PWR06
+L VCC #PWR14
 U 1 1 4ED6BA8E
 P 4550 1350
-F 0 "#PWR06" H 4550 1450 30  0001 C CNN
+F 0 "#PWR14" H 4550 1450 30  0001 C CNN
 F 1 "VCC" H 4550 1450 30  0000 C CNN
 F 2 "" H 4550 1350 60  0001 C CNN
@@
 $EndComp
 $Comp
-L GND #PWR07
+L GND #PWR25
 U 1 1 4ED6AF1D
 P 7500 6750
-F 0 "#PWR07" H 7500 6750 30  0001 C CNN
+F 0 "#PWR25" H 7500 6750 30  0001 C CNN
 F 1 "GND" H 7500 6680 30  0001 C CNN
 F 2 "" H 7500 6750 60  0001 C CNN
@@
 $EndComp
 $Comp
-L GND #PWR08
+L GND #PWR16
 U 1 1 4ED6A667
 P 4600 6450
-F 0 "#PWR08" H 4600 6450 30  0001 C CNN
+F 0 "#PWR16" H 4600 6450 30  0001 C CNN
 F 1 "GND" H 4600 6380 30  0001 C CNN
 F 2 "" H 4600 6450 60  0001 C CNN
@@
 $EndComp
 $Comp
-L GND #PWR09
+L GND #PWR11
 U 1 1 4ED6A5D7
 P 4350 6450
-F 0 "#PWR09" H 4350 6450 30  0001 C CNN
+F 0 "#PWR11" H 4350 6450 30  0001 C CNN
 F 1 "GND" H 4350 6380 30  0001 C CNN
 F 2 "" H 4350 6450 60  0001 C CNN
@@
 $EndComp
 $Comp
-L GND #PWR010
+L GND #PWR7
 U 1 1 4ED6A418
 P 3400 5350
-F 0 "#PWR010" H 3400 5350 30  0001 C CNN
+F 0 "#PWR7" H 3400 5350 30  0001 C CNN
 F 1 "GND" H 3400 5280 30  0001 C CNN
 F 2 "" H 3400 5350 60  0001 C CNN
@@
 $EndComp
 $Comp
-L VCC #PWR011
+L VCC #PWR17
 U 1 1 4EB30C92
 P 5550 1350
-F 0 "#PWR011" H 5550 1450 30  0001 C CNN
+F 0 "#PWR17" H 5550 1450 30  0001 C CNN
 F 1 "VCC" H 5550 1450 30  0000 C CNN
 F 2 "" H 5550 1350 60  0001 C CNN
@@
 $EndComp
 $Comp
-L VCC #PWR012
+L VCC #PWR19
 U 1 1 4EB30C91
 P 5650 1350
-F 0 "#PWR012" H 5650 1450 30  0001 C CNN
+F 0 "#PWR19" H 5650 1450 30  0001 C CNN
 F 1 "VCC" H 5650 1450 30  0000 C CNN
 F 2 "" H 5650 1350 60  0001 C CNN
@@
 $EndComp
 $Comp
-L VCC #PWR013
+L VCC #PWR22
 U 1 1 4EB30C90
 P 5850 1350
-F 0 "#PWR013" H 5850 1450 30  0001 C CNN
+F 0 "#PWR22" H 5850 1450 30  0001 C CNN
 F 1 "VCC" H 5850 1450 30  0000 C CNN
 F 2 "" H 5850 1350 60  0001 C CNN
@@
 $EndComp
 $Comp
-L VCC #PWR014
+L VCC #PWR24
 U 1 1 4EB30C8B
 P 5950 1350
-F 0 "#PWR014" H 5950 1450 30  0001 C CNN
+F 0 "#PWR24" H 5950 1450 30  0001 C CNN
 F 1 "VCC" H 5950 1450 30  0000 C CNN
 F 2 "" H 5950 1350 60  0001 C CNN
@@
 $EndComp
 $Comp
-L GND #PWR015
+L GND #PWR2
 U 1 1 4EB2CF09
 P 1250 2050
-F 0 "#PWR015" H 1250 2050 30  0001 C CNN
+F 0 "#PWR2" H 1250 2050 30  0001 C CNN
 F 1 "GND" H 1250 1980 30  0001 C CNN
 F 2 "" H 1250 2050 60  0001 C CNN
@@
 $EndComp
 $Comp
-L VCC #PWR016
+L VCC #PWR1
 U 1 1 4EB2CED6
 P 1250 900
-F 0 "#PWR016" H 1250 1000 30  0001 C CNN
+F 0 "#PWR1" H 1250 1000 30  0001 C CNN
 F 1 "VCC" H 1250 1000 30  0000 C CNN
 F 2 "" H 1250 900 60  0001 C CNN
@@
 $EndComp
 $Comp
-L C C6
+L C C5
 U 1 1 4EB2CECC
 P 2150 1450
-F 0 "C6" H 2200 1550 50  0000 L CNN
+F 0 "C5" H 2200 1550 50  0000 L CNN
 F 1 "100n" H 2200 1350 50  0000 L CNN
 F 2 "" H 2150 1450 60  0001 C CNN
@@
 $EndComp
 $Comp
-L C C5
+L C C4
 U 1 1 4EB2CECA
 P 1850 1450
-F 0 "C5" H 1900 1550 50  0000 L CNN
+F 0 "C4" H 1900 1550 50  0000 L CNN
 F 1 "100n" H 1900 1350 50  0000 L CNN
 F 2 "" H 1850 1450 60  0001 C CNN
@@
 $EndComp
 $Comp
-L GND #PWR017
+L GND #PWR23
 U 1 1 4E99C40C
 P 5900 6450
-F 0 "#PWR017" H 5900 6450 30  0001 C CNN
+F 0 "#PWR23" H 5900 6450 30  0001 C CNN
 F 1 "GND" H 5900 6380 30  0001 C CNN
 F 2 "" H 5900 6450 60  0001 C CNN
@@
 $EndComp
 $Comp
-L GND #PWR018
+L GND #PWR21
 U 1 1 4E99C40B
 P 5800 6450
-F 0 "#PWR018" H 5800 6450 30  0001 C CNN
+F 0 "#PWR21" H 5800 6450 30  0001 C CNN
 F 1 "GND" H 5800 6380 30  0001 C CNN
 F 2 "" H 5800 6450 60  0001 C CNN
@@
 $EndComp
 $Comp
-L GND #PWR019
+L GND #PWR20
 U 1 1 4E99C407
 P 5700 6450
-F 0 "#PWR019" H 5700 6450 30  0001 C CNN
+F 0 "#PWR20" H 5700 6450 30  0001 C CNN
 F 1 "GND" H 5700 6380 30  0001 C CNN
 F 2 "" H 5700 6450 60  0001 C CNN
@@
 $EndComp
 $Comp
-L GND #PWR020
+L GND #PWR18
 U 1 1 4E99C403
 P 5600 6450
-F 0 "#PWR020" H 5600 6450 30  0001 C CNN
+F 0 "#PWR18" H 5600 6450 30  0001 C CNN
 F 1 "GND" H 5600 6380 30  0001 C CNN
 F 2 "" H 5600 6450 60  0001 C CNN
@@
 $EndComp
 $Comp
-L GND #PWR021
+L GND #PWR8
 U 1 1 4E99B659
 P 3550 3850
-F 0 "#PWR021" H 3550 3850 30  0001 C CNN
+F 0 "#PWR8" H 3550 3850 30  0001 C CNN
 F 1 "GND" H 3550 3780 30  0001 C CNN
 F 2 "" H 3550 3850 60  0001 C CNN
@@
 $EndComp
 $Comp
-L GND #PWR022
+L GND #PWR13
 U 1 1 4E99B657
 P 4450 3850
-F 0 "#PWR022" H 4450 3850 30  0001 C CNN
+F 0 "#PWR13" H 4450 3850 30  0001 C CNN
 F 1 "GND" H 4450 3780 30  0001 C CNN
 F 2 "" H 4450 3850 60  0001 C CNN
@@
 $EndComp
 $Comp
-L GND #PWR023
+L GND #PWR12
 U 1 1 4E99B655
 P 4450 3850
-F 0 "#PWR023" H 4450 3850 30  0001 C CNN
+F 0 "#PWR12" H 4450 3850 30  0001 C CNN
 F 1 "GND" H 4450 3780 30  0001 C CNN
 F 2 "" H 4450 3850 60  0001 C CNN
@@
 $EndComp
 $Comp
-L C C4
+L C C6
 U 1 1 4E99B63E
 P 3550 3450
-F 0 "C4" H 3600 3550 50  0000 L CNN
+F 0 "C6" H 3600 3550 50  0000 L CNN
 F 1 "22p" H 3600 3350 50  0000 L CNN
 F 2 "" H 3550 3450 60  0001 C CNN
@@
 	8100 5450 8200 5550
 $Comp
-L DTSM-6 S1
+L DTSM-6 S46
 U 1 1 50440A9A
 P 3250 2300
-F 0 "S1" V 2965 2200 50  0000 L BNN
+F 0 "S46" V 2965 2200 50  0000 L BNN
 F 1 "DTSM-6" V 3065 2425 50  0000 L BNN
 F 2 "switch-tact-DTSM-6" H 3250 2450 50  0001 C CNN
@@
 	3450 5850 3200 5850
 $Comp
-L USBMINI_B05 J2
+L USBMINI_B05 J1
 U 1 1 53B498A4
 P 3000 5950
-F 0 "J2" H 2925 6250 60  0000 C CNN
+F 0 "J1" H 2925 6250 60  0000 C CNN
 F 1 "USBMINI_B05" H 2950 5600 60  0001 C CNN
 F 2 "" H 3000 5950 60  0000 C CNN
@@
 $EndComp
 $Comp
-L GND #PWR024
+L GND #PWR5
 U 1 1 53B49A83
 P 3300 6300
-F 0 "#PWR024" H 3300 6300 30  0001 C CNN
+F 0 "#PWR5" H 3300 6300 30  0001 C CNN
 F 1 "GND" H 3300 6230 30  0001 C CNN
 F 2 "" H 3300 6300 60  0001 C CNN
@@
 Main USB
 $Comp
-L VCC #PWR025
+L VCC #PWR6
 U 1 1 53B530D7
 P 3400 4650
-F 0 "#PWR025" H 3400 4750 30  0001 C CNN
+F 0 "#PWR6" H 3400 4750 30  0001 C CNN
 F 1 "VCC" H 3400 4750 30  0000 C CNN
 F 2 "" H 3400 4650 60  0001 C CNN
