File: pcb/revB/ma42_PCB_revB/matrix.sch (KiCad schematic (older format))
At the start: 88 parts

Commit message: working on revB
Parts:
- added D29: 1N4148, symbol DIODE
- added S29: MX1A, symbol MX1A
- renumbered D21 to D20, D22 to D21, D23 to D22, D25 to D23, D26 to D24, D27 to D25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
Connections:
- wire segments 148 -> 151
